File: eda/mouse-jiggler-pwm.sch (KiCad schematic (older format))
At the start: 16 parts

Commit message: pcb footprint layout
Parts:
- removed OUT: J?, symbol Connector:Screw_Terminal_01x02
- added J2: Screw_Terminal_01x02, TerminalBlock:TerminalBlock_bornier-2_P5.08mm, symbol Connector:Screw_Terminal_01x02
- C1: renamed from C?; value CAP -> 10n; footprint (none) -> Capacitor_THT:C_Disc_D3.8mm_W2.6mm_P2.50mm
- C2: renamed from C?; value CAP -> 0.1u; footprint (none) -> Capacitor_THT:C_Disc_D3.8mm_W2.6mm_P2.50mm
- D3: renamed from D?; value LED -> RED; footprint (none) -> LED_THT:LED_D5.0mm
- J1: renamed from J?; footprint (none) -> TerminalBlock:TerminalBlock_bornier-2_P5.08mm
- Q1: renamed from Q?; footprint TO254P483X1016X1994-3P -> IRFZ44NPBF:TO254P483X1016X1994-3P; symbol IRFZ44NPBF:IRFZ44NPBF -> mouse-jiggler-pwm-rescue:IRFZ44NPBF-IRFZ44NPBF
- R1, R3, R4: renamed from R?; value R_US -> 1K; footprint (none) -> Resistor_THT:R_Axial_DIN0207_L6.3mm_D2.5mm_P10.16mm_Horizontal
- R2: renamed from R?; value R_US -> 220; footprint (none) -> Resistor_THT:R_Axial_DIN0207_L6.3mm_D2.5mm_P10.16mm_Horizontal
- RV1: renamed from RV?; value R_POT_US -> 100K; footprint (none) -> Potentiometer_THT:Potentiometer_Alps_RK163_Single_Horizontal
- SW1: renamed from SW?; footprint (none) -> toggle switch:SW_Toggle_Blue_wSlots
- U1: renamed from U?; footprint Package_DIP:DIP-8_W7.62mm -> Package_DIP:DIP-8_W7.62mm_Socket
- gave numbers to parts that had none: 3
Connections:
- net at D3.1 (K), D4.1 (K), R1.1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: now also U1.8 (VCC), J2.1 (Pin_1); no longer U1.5 (CV)
- net at D4.2 (A), Q1.2: now also J2.2 (Pin_2)
- net at C1.1, RV1.2, U1.2 (TR): now also U1.6 (THR); no longer U1.7 (DIS)
- net at D1.2 (A), D2.1 (K), R1.2: now also U1.7 (DIS); no longer U1.6 (THR)
- net at C2.1: now also U1.5 (CV); no longer U1.8 (VCC)
Other:
- moved on the sheet: C1, C2

Commit message: fix toggle switch footprint and generate gerber
Parts:
- SW1: footprint toggle switch:SW_Toggle_Blue_wSlots -> 100SP1T1B4M2QE-Switch:100SP1T1B4M2QE
Changed lines of the file:
@@
 F 0 "SW1" H 3650 3035 50  0000 C CNN
 F 1 "SW_DPDT_x2" H 3650 2944 50  0000 C CNN
-F 2 "toggle switch:SW_Toggle_Blue_wSlots" H 3650 2750 50  0001 C CNN
+F 2 "100SP1T1B4M2QE-Switch:100SP1T1B4M2QE" H 3650 2750 50  0001 C CNN
 F 3 "~" H 3650 2750 50  0001 C CNN
 	1    3650 2750
